File: PCB_rev_A4/Replicape_A4.sch (EAGLE design)
At the start: 188 parts, among them P8 F-2X23-, P9 F-2X23-, Q1 AON6758, Q2 AON6758, Q3 AON6758, Q4 NIF5002, Q5 NIF5002, Q6 NIF5002, U1 SN74AHC595PW, U10 RT8268, U11 PCA9685PW, U12 DAC088S085, U13 DRV8825PWP, U14 DRV8825PWP, U15 DRV8825PWP, U16 DRV8825PWP, U17 DRV8825PWP, U18 CAT24C256, U2 SN74AHC595PW, U3 SN74AHC595PW, U4 SN74AHC595PW, U5 SN74AHC595PW, U6 MCP16321, U7 MCP1402, U8 MCP1402, U9 MCP1402, X1 22-05-7028-02, X10 22-05-7028-02, X11 22-05-7028-02, X12 22-05-7038-03, X13 22-05-7028-02, X14 22-05-7048-04, X15 22-05-7048-04, X16 22-05-7048-04, X17 22-05-7048-04, X18 22-05-7048-04, X19 22-05-7028-02, X2 MSTBA4, X20 MSTBA4, X21 MSTBA2, X23 22-05-7028-02, X3 MSTBA2, X4 22-05-7028-02, X5 22-05-7028-02, X6 22-05-7028-02, X7 22-05-7038-03, X8 22-05-7038-03, X9 22-05-7038-03

Commit message: Changed the pullup VDD from 5V to 3.3V
Parts:
- added C60: 0.47uF, rcl:C-EUC0402
- F1: value 3557 -> FUSE3557; device SparkFun:3557 -> fuse:FUSE3557
Connections:
- net +3V3: now also C60.1, R49.2, R50.2, R51.2, R52.2, R53.2, R54.2, X12-1.S
- net GND: now also C60.2, U6.PGND; no longer U6.PGND@14, U6.PGND@15
- net N$114: no longer Q6.D@1
- net N$115: no longer Q5.D@1
- net N$116: no longer Q4.D@1
- net SW: now also U6.SW; no longer U6.SW@1, U6.SW@12, U6.SW@13, U6.SW@16
- net SYS_5V: no longer R49.2, R50.2, R51.2, R52.2, R53.2, R54.2, X12-1.S
- net VDD_IN: now also F1.2, U6.VIN; no longer F1.3, F1.4, U6.VIN@11, U6.VIN@2, U6.VIN@3
- net VIN: no longer F1.2

Commit message: Added a cap across 5V for stability.
Parts:
- added C61: 100uF, rcl:CPOL-EU140CLH-0810
Connections:
- net GND: now also C61.-
- net VDD_5V: now also C61.+
Changed lines of the file:
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@@
 <?xml version="1.0" encoding="utf-8"?>
 <!DOCTYPE eagle SYSTEM "eagle.dtd">
-<eagle version="6.1">
+<eagle version="6.5.0">
 <drawing>
 <settings>
@@
 <part name="GND81" library="supply1" deviceset="GND" device=""/>
 <part name="F1" library="fuse" deviceset="FUSE" device="3557"/>
+<part name="C61" library="rcl" deviceset="CPOL-EU" device="140CLH-0810" value="100uF"/>
+<part name="GND82" library="supply1" deviceset="GND" device=""/>
 </parts>
 <sheets>
@@
 <instance part="C60" gate="G$1" x="599.44" y="162.56" rot="MR0"/>
 <instance part="GND81" gate="1" x="599.44" y="154.94" rot="MR0"/>
+<instance part="C61" gate="G$1" x="142.24" y="76.2"/>
+<instance part="GND82" gate="1" x="142.24" y="63.5"/>
 </instances>
 <busses>
@@
 <pinref part="C60" gate="G$1" pin="2"/>
 <pinref part="GND81" gate="1" pin="GND"/>
+</segment>
+<segment>
+<pinref part="C61" gate="G$1" pin="-"/>
+<wire x1="142.24" y1="71.12" x2="142.24" y2="66.04" width="0.1524" layer="91"/>
+<pinref part="GND82" gate="1" pin="GND"/>
 </segment>
 </net>
@@
 <pinref part="U6" gate="G$1" pin="VFB"/>
 <pinref part="5V" gate="G$1" pin="TP"/>
-</segment>
-<segment>
+<pinref part="C61" gate="G$1" pin="+"/>
+<wire x1="142.24" y1="86.36" x2="142.24" y2="78.74" width="0.6096" layer="91"/>
+<junction x="142.24" y="86.36"/>
+</segment>
+<segment>

Commit message: Added a series resistor for Cboost to limit noise
Parts:
- removed C61: 100uF, rcl:CPOL-EU140CLH-0810
- added R58: 100R, rcl:R-EU_R0402
Connections:
- new net N$1: C51.1, R58.1
- net GND: no longer C61.-
- net N$128: now also R58.2; no longer C51.1
- net VDD_5V: no longer C61.+
Other:
- moved on the sheet: C51
Changed lines of the file:
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@@
 <part name="GND81" library="supply1" deviceset="GND" device=""/>
 <part name="F1" library="fuse" deviceset="FUSE" device="3557"/>
-<part name="C61" library="rcl" deviceset="CPOL-EU" device="140CLH-0810" value="100uF"/>
-<part name="GND82" library="supply1" deviceset="GND" device=""/>
+<part name="R58" library="rcl" deviceset="R-EU_" device="R0402" value="100R"/>
 </parts>
 <sheets>
@@
 <instance part="GND29" gate="1" x="119.38" y="76.2"/>
 <instance part="GND30" gate="1" x="71.12" y="53.34"/>
-<instance part="C51" gate="G$1" x="83.82" y="96.52" rot="R90"/>
+<instance part="C51" gate="G$1" x="88.9" y="96.52" rot="R90"/>
 <instance part="R41" gate="G$1" x="134.62" y="76.2" rot="R90"/>
 <instance part="L1" gate="G$1" x="104.14" y="86.36" rot="R90"/>
@@
 <instance part="C60" gate="G$1" x="599.44" y="162.56" rot="MR0"/>
 <instance part="GND81" gate="1" x="599.44" y="154.94" rot="MR0"/>
-<instance part="C61" gate="G$1" x="142.24" y="76.2"/>
-<instance part="GND82" gate="1" x="142.24" y="63.5"/>
+<instance part="R58" gate="G$1" x="78.74" y="96.52" rot="R180"/>
 </instances>
 <busses>
@@
 <pinref part="GND81" gate="1" pin="GND"/>
 </segment>
-<segment>
-<pinref part="C61" gate="G$1" pin="-"/>
-<wire x1="142.24" y1="71.12" x2="142.24" y2="66.04" width="0.1524" layer="91"/>
-<pinref part="GND82" gate="1" pin="GND"/>
-</segment>
 </net>
 <net name="N$114" class="0">
@@
 <pinref part="U6" gate="G$1" pin="VFB"/>
 <pinref part="5V" gate="G$1" pin="TP"/>
-<pinref part="C61" gate="G$1" pin="+"/>
-<wire x1="142.24" y1="86.36" x2="142.24" y2="78.74" width="0.6096" layer="91"/>
-<junction x="142.24" y="86.36"/>
 </segment>
 <segment>
@@
 <segment>
 <wire x1="73.66" y1="93.98" x2="73.66" y2="96.52" width="0.1524" layer="91"/>
-<wire x1="73.66" y1="96.52" x2="81.28" y2="96.52" width="0.1524" layer="91"/>
 <pinref part="U6" gate="G$1" pin="BOOST"/>
-<pinref part="C51" gate="G$1" pin="1"/>
+<pinref part="R58" gate="G$1" pin="2"/>
 </segment>
 </net>
@@
 <net name="SW" class="0">
 <segment>
-<wire x1="91.44" y1="86.36" x2="93.98" y2="86.36" width="0.6096" layer="91"/>
-<wire x1="88.9" y1="96.52" x2="93.98" y2="96.52" width="0.1524" layer="91"/>
-<wire x1="93.98" y1="96.52" x2="93.98" y2="86.36" width="0.1524" layer="91"/>
-<wire x1="93.98" y1="86.36" x2="99.06" y2="86.36" width="0.6096" layer="91"/>
-<junction x="93.98" y="86.36"/>
+<wire x1="91.44" y1="86.36" x2="96.52" y2="86.36" width="0.6096" layer="91"/>
+<wire x1="93.98" y1="96.52" x2="96.52" y2="96.52" width="0.1524" layer="91"/>
+<wire x1="96.52" y1="96.52" x2="96.52" y2="86.36" width="0.1524" layer="91"/>
+<wire x1="96.52" y1="86.36" x2="99.06" y2="86.36" width="0.6096" layer="91"/>
+<junction x="96.52" y="86.36"/>
 <pinref part="U6" gate="G$1" pin="SW"/>
 <pinref part="C51" gate="G$1" pin="2"/>
@@
 </segment>
 </net>
+<net name="N$1" class="0">
+<segment>
+<pinref part="C51" gate="G$1" pin="1"/>
+<pinref part="R58" gate="G$1" pin="1"/>
+<wire x1="86.36" y1="96.52" x2="83.82" y2="96.52" width="0.1524" layer="91"/>
+</segment>
+</net>
