File: PCB_rev_A4A/Replicape_A4A.sch (EAGLE design)
At the start: 190 parts, among them P8 F-2X23-, P9 F-2X23-, Q1 AON6758, Q2 AON6758, Q3 AON6758, Q4 NIF5002, Q5 NIF5002, Q6 NIF5002, U1 SN74AHC595PW, U10 RT8268, U11 PCA9685PW, U12 DAC088S085, U13 DRV8825PWP, U14 DRV8825PWP, U15 DRV8825PWP, U16 DRV8825PWP, U17 DRV8825PWP, U18 CAT24C256, U2 SN74AHC595PW, U3 SN74AHC595PW, U4 SN74AHC595PW, U5 SN74AHC595PW, U6 MCP16321, U7 MCP1402, U8 MCP1402, U9 MCP1402, X1 22-05-7028-02, X10 22-05-7028-02, X11 22-05-7028-02, X12 22-05-7038-03, X13 22-05-7028-02, X14 22-05-7048-04, X15 22-05-7048-04, X16 22-05-7048-04, X17 22-05-7048-04, X18 22-05-7048-04, X19 22-05-7028-02, X2 MSTBA4, X20 MSTBA4, X21 MSTBA2, X23 22-05-7028-02, X3 MSTBA2, X4 22-05-7028-02, X5 22-05-7028-02, X6 22-05-7028-02, X7 22-05-7038-03, X8 22-05-7038-03, X9 22-05-7038-03

Commit message: Updated A4A
Parts:
- added EXPAND: EXPAND, con-lstb:MA05-2
- added U$3: CC-BY-SA, cc-by-sa:CC-BY-SA
Connections:
- net STEP1_X renamed A1_X
- net STEP2_X renamed A2_X
- removed net STEP3_X: U13.BOUT1, X14-2.S
- removed net STEP3_Z: U15.BOUT1, X16-2.S
- removed net STEP4_X: U13.BOUT2, X14-1.S
- removed net STEP4_Y: U14.BOUT2, X15-1.S
- removed net STEP4_Z: U15.BOUT2, X16-1.S
- new net B1_X: U13.BOUT1, X14-1.S
- new net FAN4: EXPAND.9, U11.LED14
- new net FAN5: EXPAND.8, U11.LED15
- new net FAN6: EXPAND.7, U11.LED7
- new net HEATER_EXT3: EXPAND.5, U11.LED11
- new net HEATER_EXT4: EXPAND.3, U11.LED12
- new net HEATER_EXT5: EXPAND.1, U11.LED13
- new net N$2: U13.BOUT2, X14-2.S
- new net N$3: U14.BOUT2, X15-2.S
- new net N$4: U15.BOUT1, X16-1.S
- new net N$5: U15.BOUT2, X16-2.S
- new net SER6: EXPAND.10, U5.QH_2
- new net VREF_EXT3: EXPAND.2, U12.P$13-VOUTF
- new net VREF_EXT4: EXPAND.4, U12.P$12-VOUTG
- new net VREF_EXT5: EXPAND.6, U12.P$11-VOUTH
- net STEP3_EXT1: now also X17-1.S; no longer X17-2.S
- net STEP3_EXT2: now also X18-1.S; no longer X18-2.S
- net STEP3_Y: now also X15-1.S; no longer X15-2.S
- net STEP4_EXT1: now also X17-2.S; no longer X17-1.S
- net STEP4_EXT2: now also X18-2.S; no longer X18-1.S
- net SYS_5V: no longer P9.7
Other:
- moved on the sheet: X14-1, X14-2, X15-1, X15-2, X16-1, X16-2, X17-1, X17-2, X18-1, X18-2
